File: Projeto_IA/Projeto_IA/PCB_IA/PCB_IA.kicad_pcb (KiCad board)
At the start: 2 copper layers, 37.5 x 80 mm, 6 parts, among them U1 ESP32-S2, U2 LSM6DS3, Y1 Crystal_Small

Commit message: Commitando versão nova de placa
Parts:
- added R1: 0, Resistor_SMD:R_01005_0402Metric, F.Cu at (115.2, 66.5)
- added SW1: SW_Nidec_CAS-120A1, Button_Switch_SMD:Nidec_Copal_CAS-120A, F.Cu at (101.2, 107.8)
- added SW2: SW_Nidec_CAS-120A1, Button_Switch_SMD:Nidec_Copal_CAS-120A, F.Cu at (117.8, 104.5)
- added Y2: ASDMB-xxxMHz, Oscillator:Oscillator_SMD_Abracon_ASDMB-4Pin_2.5x2.0mm, F.Cu at (100.8, 67.7)
- moved Y1 30.1 mm to (125.3, 105.8)
- moved C2 21.1 mm to (128.6, 70.7), turned to 0 degrees
- moved C1 7.16 mm to (100.9, 81.8), turned to 0 degrees
Connections:
- C1 pad 1: /POWER_BAT -> /ACC_VDD
- U1 pad 6: unconnected-(U1-GPIO1-Pad6) -> /OSC_INIT
- U1 pad 7: unconnected-(U1-GPIO2-Pad7) -> /ACC_INIT
- U2 pad 8: /POWER_BAT -> /ACC_VDD
Routing:
- net /SIGNAL_CRYSP: track 21.4 -> 6.56 mm, vias 2 -> 1
- net /SIGNAL_CRYSN: track 18.3 -> 6.14 mm, vias 2 -> 0
