File: Projeto_IA/Projeto_IA/PCB_IA/PCB_IA.kicad_sch (KiCad schematic)
At the start: 6 parts, among them U1 ESP32-S2, U2 LSM6DS3, Y1 Crystal_Small

Commit message: Commitando versão nova de placa
Parts:
- added R1: 0, Resistor_SMD:R_01005_0402Metric, symbol Device:R
- added SW1, SW2: SW_Nidec_CAS-120A1, Button_Switch_SMD:Nidec_Copal_CAS-120A, symbol Switch:SW_Nidec_CAS-120A1
- added Y2: ASDMB-xxxMHz, Oscillator:Oscillator_SMD_Abracon_ASDMB-4Pin_2.5x2.0mm, symbol Oscillator:ASDMB-xxxMHz
Connections:
- net ACC_CLK: now also R1.2
- net GND: now also Y2.2 (GND)
- net POWER_BAT: no longer C1.1, U2.8 (VDD)
- net OSC_INIT: now reaches U1.6 (GPIO1)
- net OSC_INIT: now also SW1.2 (B)
- net ACC_INIT: now reaches U1.7 (GPIO2)
- net ACC_INIT: now also SW2.2 (B)
- new net ACC_CLK_EXT: R1.1, Y2.3 (Out)
- new net ACC_VDD: C1.1, SW2.3 (A), U2.8 (VDD), Y2.4 (VDD)
- new net OSC_VDD: SW1.3 (A)
- no-connect marks 13 -> 15
Other:
- moved on the sheet: Y1
